File: kicadfiles/eava55.kicad_pcb (KiCad board)
At the start: 2 copper layers, 305 x 94.7 mm, 164 parts, among them J1 Conn_01x04_Pin, SW1 SW_DPST_x2, SW2 SW_DPST_x2, U1 XC6206PxxxMR, U2 SRV05-4, U3 STM32F072CBTx, U4 TLV74318PDBVR, U5 PMW3360DM-T2QU

Commit message: updated pcb edge cut
Parts:
- moved D71 6.65 mm to (307.5, 105.4), turned to 0 degrees
Routing:
- net ROW4: track 334.8 -> 325.9 mm
- net Net-(D71-A): track 13.0 -> 17.7 mm
- net COL13: track 70.6 -> 71.3 mm
- net COL14: track 58.2 -> 59.0 mm
- net COL15: track 84.6 -> 85.3 mm
- net GND: vias 21 -> 24
Other:
- board size 305 x 94.7 mm -> 301.8 x 93.5 mm
